File: kicad/boost_sequencer.kicad_pcb (KiCad board)
At the start: 2 copper layers, 59 x 40 mm, 70 parts, among them J1 Conn_01x07_Female, J2 Conn_01x03_Male, J3 Conn_01x04_Female, J4 Conn_01x07_Female, Q1 PDTC144E, Q10 BC817, Q11 BC817, Q12 BC807, Q13 BC807, Q14 *N, Q2 PDTC144E, Q3 PDTC144E, Q4 *P, Q5 *P, Q6 *N, Q7 *N, Q8 PDTC144E, Q9 *P, U1 LM317_SOT-223, U2 ATtiny416-S

Commit message: Fixed error: TN/TP were interchanged
Other:
- net class Default removed
